File: board/board.kicad_pcb (KiCad board)
At the start: 2 copper layers, 21 x 13 mm, 1 part

Commit message: initial
Parts:
- added C1: 1uF, Capacitor_SMD:C_0603_1608Metric, F.Cu at (153.8, 101.2)
- added C2: 10uF, Capacitor_SMD:C_0603_1608Metric, F.Cu at (155.2, 101.2)
- added C3: 10uF, Capacitor_SMD:C_0603_1608Metric, F.Cu at (147.3, 98.2)
- added C4: 10uF, Capacitor_SMD:C_0603_1608Metric, F.Cu at (145.8, 98.2)
- added C5: 1uF, Capacitor_SMD:C_0603_1608Metric, F.Cu at (148.8, 98.2)
- added J1: 003_power, on_edge:on_edge_2x05_device, F.Cu at (140.0, 96.5)
- added J2: 003_power, on_edge:on_edge_2x05_host, F.Cu at (161.0, 96.5)
- added J3: Conn_01x03_Male, Connector_PinHeader_2.54mm:PinHeader_1x03_P2.54mm_Vertical, F.Cu at (146.1, 101.5)
- added R1: 0R, Resistor_SMD:R_0603_1608Metric, B.Cu at (146.6, 98.0)
- added R2: 0R, Resistor_SMD:R_0603_1608Metric, B.Cu at (154.4, 98.1)
- added U1: LD39200PU33R, b121:SON95P300X300X100-7N, F.Cu at (151.7, 97.9)
- LOGO1: moved to B.Cu
- moved LOGO1 5.95 mm to (150.8, 93.1), turned to 180 degrees
Routing:
- net /ldo/GND: track 0.00 -> 51.8 mm, vias 0 -> 16
- net /ldo/5v: track 0.00 -> 25.3 mm, vias 0 -> 2
- net Net-(J1-Pad4): track 0.00 -> 19.2 mm, vias 0 -> 2
- net Net-(J1-Pad8): track 0.00 -> 18.1 mm
- net Net-(J1-Pad7): track 0.00 -> 18.0 mm
- net Net-(J1-Pad3): track 0.00 -> 17.9 mm, vias 0 -> 2
- net Net-(J1-Pad5): track 0.00 -> 17.6 mm, vias 0 -> 2
- net Net-(J1-Pad2): track 0.00 -> 17.3 mm, vias 0 -> 2
- net Net-(J1-Pad6): track 0.00 -> 16.5 mm
- net /ldo/3.3v: track 0.00 -> 13.5 mm, vias 0 -> 1
- net /ldo/EN: track 0.00 -> 7.83 mm, vias 0 -> 1
- net Net-(J1-Pad9): track 0.00 -> 3.51 mm
- net Net-(J2-Pad9): track 0.00 -> 3.49 mm
- added copper zone on B.Cu, net /ldo/GND
- added copper zone on F.Cu, net /ldo/GND
Other:
- outline, holes or cut-outs redrawn
- board text added: "enable"
- board text added: "osf.003"
- board text added: "osf.b121.v1.0"
